Commit message: Adding bondgraphs.jl

File: niryo_one_description/urdf/v1/niryo_one.urdf (robot description, URDF)
Before this commit: robot niryo_one, 9 links, 8 joints
Links:
- link arm_link: geometry collision mesh filename=/home/carson/research/SmartManufacturing/SmartManufacturing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; visual mesh filename=/home/carson/research/SmartManufacturing/SmartManufacturing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
- link base_link: geometry collision mesh filename=/home/carson/research/SmartManufacturing/SmartManufacturing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; visual mesh filename=/home/carson/research/SmartManufacturing/SmartManufacturing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
- link elbow_link: geometry collision mesh filename=/home/carson/research/SmartManufacturing/SmartManufacturing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; visual mesh filename=/home/carson/research/SmartManufacturing/SmartManufacturing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
- link forearm_link: geometry collision mesh filename=/home/carson/research/SmartManufacturing/SmartManufacturing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; visual mesh filename=/home/carson/research/SmartManufacturing/SmartManufacturing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
- link hand_link: geometry collision mesh filename=/home/carson/research/SmartManufacturing/SmartManufacturing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; visual mesh filename=/home/carson/research/SmartManufacturing/SmartManufacturing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
- link shoulder_link: geometry collision mesh filename=/home/carson/research/SmartManufacturing/SmartManufacturing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; visual mesh filename=/home/carson/research/SmartManufacturing/SmartManufacturing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
- link wrist_link: geometry collision mesh filename=/home/carson/research/SmartManufacturing/SmartManufacturing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; visual mesh filename=/home/carson/research/SmartManufacturing/SmartManufacturing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

Commit message: Added Presentation Notebook

File: niryo_one_description/urdf/v1/niryo_one.urdf (robot description, URDF)
Before this commit: robot niryo_one, 9 links, 8 joints
Links:
- link arm_link: geometry collision mesh filename=PATH/niryo_one_description/meshes/v1/stl/arm_link.stl; visual mesh filename=PATH/niryo_one_description/meshes/v1/stl/arm_link.stl
- link base_link: geometry collision mesh filename=PATH/niryo_one_description/meshes/v1/stl/base_link.stl; visual mesh filename=PATH/niryo_one_description/meshes/v1/stl/base_link.stl
- link elbow_link: geometry collision mesh filename=PATH/niryo_one_description/meshes/v1/stl/elbow_link.stl; visual mesh filename=PATH/niryo_one_description/meshes/v1/stl/elbow_link.stl
- link forearm_link: geometry collision mesh filename=PATH/niryo_one_description/meshes/v1/stl/forearm_link.stl; visual mesh filename=PATH/niryo_one_description/meshes/v1/stl/forearm_link.stl
- link hand_link: geometry collision mesh filename=PATH/niryo_one_description/meshes/v1/stl/hand_link.stl; visual mesh filename=PATH/niryo_one_description/meshes/v1/stl/hand_link.stl
- link shoulder_link: geometry collision mesh filename=PATH/niryo_one_description/meshes/v1/stl/shoulder_link.stl; visual mesh filename=PATH/niryo_one_description/meshes/v1/stl/shoulder_link.stl
- link wrist_link: geometry collision mesh filename=PATH/niryo_one_description/meshes/v1/stl/wrist_link.stl; visual mesh filename=PATH/niryo_one_description/meshes/v1/stl/wrist_link.stl
